Commit message: add lidar

File: models/basic_mobile_robot/model.sdf.xacro (robot description, xacro)
@@ -2,290 +2,367 @@
 <sdf version="1.5">
   <model name="basic_mobile_bot">
-  <static>false</static>
-  <!-- ****************** ROBOT BASE FOOTPRINT ***************************  -->
-  <pose>0.0 0.0 0.0 0.0 0.0 0.0</pose>
-  <link name="base_footprint"/>
-  <!-- ********************** ROBOT BASE *********************************  -->
-  <link name="base_link">
-    <collision name="base_collision">
-      <pose>0 0 0.1 0 0 0</pose>
-      <geometry>
-        <box>
-          <size>0.70 0.39 0.20</size>
-        </box>
-      </geometry>
-    </collision>
-    <visual name="base_visual">
-      <pose>0 0 -0.05 1.5707963267949 0 3.141592654</pose>
-      <geometry>
-        <mesh>
-          <!-- <uri>model://basic_mobile_robot/meshes/robot_base.stl</uri> -->
-          <uri>file://$(find basic_mobile_robot)/models/basic_mobile_robot/meshes/robot_base.stl</uri>
-          <scale>1.0 1.0 1.0</scale>
-        </mesh>
-      </geometry>
-      <material>
-        <ambient>1.0 0.0 0.0 1.0</ambient>
-        <diffuse>1.0 0.0 0.0 1.0</diffuse>
-        <specular>0.0 0.0 0.0 1.0</specular>
-        <emissive>0.0 0.0 0.0 1.0</emissive>
-      </material>
-    </visual>
-  </link>
-  <!-- *********************** IMU SENSOR SETUP **************************  -->
-  <link name="imu_link">
-    <gravity>true</gravity>
-    <sensor name="bmb_imu" type="imu">
-      <always_on>true</always_on>
-      <update_rate>100</update_rate>
-      <visualize>true</visualize>
-      <imu>
-        <orientation>
-          <x>
-            <noise type="gaussian">
-              <mean>0.0</mean>
-              <stddev>2e-3</stddev>
-            </noise>
-          </x>
-          <y>
-            <noise type="gaussian">
-              <mean>0.0</mean>
-              <stddev>2e-3</stddev>
-            </noise>
-          </y>
-          <z>
-            <noise type="gaussian">
-              <mean>0.0</mean>
-              <stddev>2e-3</stddev>
-            </noise>
-          </z>
-        </orientation>
-        <angular_velocity>
-          <x>
-            <noise type="gaussian">
-              <mean>0.0</mean>
-              <stddev>2e-4</stddev>
-            </noise>
-          </x>
-          <y>
-            <noise type="gaussian">
-              <mean>0.0</mean>
-              <stddev>2e-4</stddev>
-            </noise>
-          </y>
-          <z>
-            <noise type="gaussian">
-              <mean>0.0</mean>
-              <stddev>2e-4</stddev>
-            </noise>
-          </z>
-        </angular_velocity>
-        <linear_acceleration>
-          <x>
-            <noise type="gaussian">
-              <mean>0.0</mean>
-              <stddev>1.7e-2</stddev>
-            </noise>
-          </x>
-          <y>
-            <noise type="gaussian">
-              <mean>0.0</mean>
-              <stddev>1.7e-2</stddev>
-            </noise>
-          </y>
-          <z>
-            <noise type="gaussian">
-              <mean>0.0</mean>
-              <stddev>1.7e-2</stddev>
-            </noise>
-          </z>
-        </linear_acceleration>
-      </imu>
-      <plugin name="basic_mobile_bot_imu" filename="libgazebo_ros_imu_sensor.so">
-        <initial_orientation_as_reference>false</initial_orientation_as_reference>
-        <frame_name>imu_link</frame_name>
-        <ros>
-          <namespace>/imu</namespace>
-          <remapping>~/out:=data</remapping>
-        </ros>
-      </plugin>
-    </sensor>
-  </link>
-  <!-- *********************** GPS SETUP *********************************  -->
-  <link name="gps_link">
-    <sensor name="bmb_gps" type="gps">
-      <always_on>true</always_on>
-      <update_rate>10.0</update_rate>
-      <gps>
-        <position_sensing>
-          <horizontal>
-            <noise type="gaussian">
-              <mean>0.0</mean>
-              <stddev>1e-2</stddev>
-            </noise>
-          </horizontal>
-          <vertical>
-            <noise type="gaussian">
-              <mean>0.0</mean>
-              <stddev>1</stddev>
-            </noise>
-          </vertical>
-        </position_sensing>
-      </gps>
-      <plugin name="basic_mobile_bot_gps" filename="libgazebo_ros_gps_sensor.so">
-        <ros>
-          <remapping>~/out:=gps/fix</remapping>
-        </ros>
-      </plugin>
-    </sensor>
-  </link>
-  <!-- *********************** DRIVE WHEELS ******************************  -->
-  <link name="drivewhl_l_link">
-    <pose>-0.221 0.23 -0.05 0 1.570796 1.570796</pose>
-    <collision name="drivewhl_l_collision">
-      <geometry>
-        <cylinder>
-          <radius>0.14</radius>
-          <length>0.06</length>
-        </cylinder>
-      </geometry>
-    </collision>
-    <visual name="drivewhl_l_visual">
-      <geometry>
-        <cylinder>
-          <radius>0.14</radius>
-          <length>0.06</length>
-        </cylinder>
-      </geometry>
-    </visual>
-  </link>
-  <link name="drivewhl_r_link">
-    <pose>-0.221 -0.23 -0.05 0 1.570796 1.570796</pose>
-    <collision name="drivewhl_r_collision">
-      <geometry>
-        <cylinder>
-          <radius>0.14</radius>
-          <length>0.06</length>
-        </cylinder>
-      </geometry>
-    </collision>
-    <visual name="drivewhl_r_visual">
-      <geometry>
-        <cylinder>
-          <radius>0.14</radius>
-          <length>0.06</length>
-        </cylinder>
-      </geometry>
-    </visual>
-  </link>
-  <!-- *********************** CASTER WHEEL ******************************  -->
-  <link name='front_caster'>
-    <pose>0.217 0 -0.1 0 0 0</pose>
-    <collision name='collision'>
-      <geometry>
-        <sphere>
-          <radius>0.09</radius>
-        </sphere>
-      </geometry>
-      <surface>
-        <friction>
-          <ode>
-            <mu>0.01</mu>
-            <mu2>0.01</mu2>
-            <slip1>1.0</slip1>
-            <slip2>1.0</slip2>
-          </ode>
-        </friction>
-      </surface>
-    </collision>
-    <visual name="front_caster_visual">
-      <geometry>
-        <sphere>
-          <radius>0.09</radius>
-        </sphere>
-      </geometry>
-    </visual>
-  </link>
-  <!-- ************************ JOINTS ***********************************  -->
-  <!-- Pose of the joint is the same as the child link frame -->
-  <!-- Axis is the axis of rotation relative to the child link frame -->
-  <joint name="base_joint" type="fixed">
-    <parent>base_footprint</parent>
-    <child>base_link</child>
-    <pose>0 0 0 0 0 0</pose>
-  </joint>
-  <joint name="drivewhl_l_joint" type="revolute">
-    <parent>base_link</parent>
-    <child>drivewhl_l_link</child>
-    <pose>0 0 0 0 0 0</pose>
-    <axis>
-      <xyz>0 0 1</xyz>
-    </axis>
-  </joint>
-  <joint name="drivewhl_r_joint" type="revolute">
-    <parent>base_link</parent>
-    <child>drivewhl_r_link</child>
-    <pose>0 0 0 0 0 0</pose>
-    <axis>
-      <xyz>0 0 1</xyz>
-    </axis>
-  </joint>
-  <joint name='caster_joint' type='fixed'>
-    <parent>base_link</parent>
-    <child>front_caster</child>
-    <pose>0 0 0 0 0 0</pose>
-  </joint>
-  <joint name="imu_joint" type="fixed">
-    <parent>base_link</parent>
-    <child>imu_link</child>
-    <pose>0 0 0 0 0 0</pose>
-  </joint>
-  <joint name="gps_joint" type="fixed">
-    <parent>base_link</parent>
-    <child>gps_link</child>
-    <pose>0 0 0 0 0 0</pose>
-  </joint>
- <!-- *********************** WHEEL ODOMETRY ***************************    -->
-  <plugin name="basic_mobile_bot_diff_drive" filename="libgazebo_ros_diff_drive.so">
-    <update_rate>30</update_rate>
-    <!-- wheels -->
-    <left_joint>drivewhl_l_joint</left_joint>
-    <right_joint>drivewhl_r_joint</right_joint>
-    <!-- kinematics -->
-    <wheel_separation>0.52</wheel_separation>
-    <wheel_diameter>0.28</wheel_diameter>
-    <!-- limits -->
-    <max_wheel_torque>20</max_wheel_torque>
-    <max_wheel_acceleration>1.0</max_wheel_acceleration>
-    <!-- Receive velocity commands on this ROS topic -->
-    <command_topic>cmd_vel</command_topic>
-    <!-- output -->
-    <!-- When false, publish no wheel odometry data to a ROS topic -->
-    <publish_odom>true</publish_odom>
-    <!-- When true, publish coordinate transform from odom to base_footprint -->
-    <!-- I usually use the robot_localization package to publish this transform -->
-    <publish_odom_tf>false</publish_odom_tf>
-    <!-- When true, publish coordinate transform from base_link to the wheels -->
-    <!-- The robot_state_publisher package is often used to publish this transform -->
-    <publish_wheel_tf>false</publish_wheel_tf>
-    <odometry_topic>odom</odometry_topic>
-    <odometry_frame>odom</odometry_frame>
-    <robot_base_frame>base_footprint</robot_base_frame>
-    <!-- Odometry source, 0 for ENCODER, 1 for WORLD, defaults to WORLD -->
-    <odometry_source>0</odometry_source>
-    <!-- Change the ROS topic we will publish the odometry data to -->
-    <ros>
-      <remapping>odom:=wheel/odometry</remapping>
-    </ros>
-  </plugin>
- <!-- *********************** JOINT STATE PUBLISHER *********************   -->
-  <plugin name="basic_mobile_bot_joint_state" filename="libgazebo_ros_joint_state_publisher.so">
-    <ros>
-      <remapping>~/out:=joint_states</remapping>
-    </ros>
-    <update_rate>30</update_rate>
-    <joint_name>drivewhl_l_joint</joint_name>
-    <joint_name>drivewhl_r_joint</joint_name>
-  </plugin>
+    <static>false</static>
+    <!-- ****************** ROBOT BASE FOOTPRINT ***************************  -->
+    <pose>0.0 0.0 0.0 0.0 0.0 0.0</pose>
+    <link name="base_footprint"/>
+    <!-- ********************** ROBOT BASE *********************************  -->
+    <link name="base_link">
+      <collision name="base_collision">
+        <pose>0 0 0.1 0 0 0</pose>
+        <geometry>
+          <box>
+            <size>0.70 0.39 0.20</size>
+          </box>
+        </geometry>
+      </collision>
+      <visual name="base_visual">
+        <pose>0 0 -0.05 1.5707963267949 0 3.141592654</pose>
+        <geometry>
+          <mesh>
+            <!-- <uri>model://basic_mobile_robot/meshes/robot_base.stl</uri> -->
+            <uri>file://$(find basic_mobile_robot)/models/basic_mobile_robot/meshes/robot_base.stl</uri>
+            <scale>1.0 1.0 1.0</scale>
+          </mesh>
+        </geometry>
+        <material>
+          <ambient>1.0 0.0 0.0 1.0</ambient>
+          <diffuse>1.0 0.0 0.0 1.0</diffuse>
+          <specular>0.0 0.0 0.0 1.0</specular>
+          <emissive>0.0 0.0 0.0 1.0</emissive>
+        </material>
+      </visual>
+    </link>
+    <!-- ****************************** LIDAR *****************************    -->
+    <link name="lidar_link">
+      <inertial>
+        <pose>0.215 0 0.13 0 0 0</pose>
+        <inertia>
+          <ixx>0.001</ixx>
+          <ixy>0.000</ixy>
+          <ixz>0.000</ixz>
+          <iyy>0.001</iyy>
+          <iyz>0.000</iyz>
+          <izz>0.001</izz>
+        </inertia>
+        <mass>0.114</mass>
+      </inertial>
+      <collision name="lidar_collision">
+        <pose>0.215 0 0.13 0 0 0</pose>
+        <geometry>
+          <cylinder>
+            <radius>0.0508</radius>
+            <length>0.18</length>
+          </cylinder>
+        </geometry>
+      </collision>
+      <visual name="lidar_visual">
+        <pose>0.215 0 0.13 0 0 0</pose>
+        <geometry>
+          <cylinder>
+            <radius>0.0508</radius>
+            <length>0.18</length>
+          </cylinder>
+        </geometry>
+        <material>
+          <ambient>0.0 0.0 0.0 1.0</ambient>
+          <diffuse>0.0 0.0 0.0 1.0</diffuse>
+          <specular>0.0 0.0 0.0 1.0</specular>
+          <emissive>0.0 0.0 0.0 1.0</emissive>
+        </material>
+      </visual>
+      <sensor name="lidar" type="ray">
+        <pose>0.215 0 0.215 0 0 0</pose>
+        <always_on>true</always_on>
+        <visualize>true</visualize>
+        <update_rate>5</update_rate>
+        <ray>
+          <scan>
+            <horizontal>
+              <samples>360</samples>
+              <resolution>1.00000</resolution>
+              <min_angle>0.000000</min_angle>
+              <max_angle>6.280000</max_angle>
+            </horizontal>
+          </scan>
+          <range>
+            <min>0.120000</min>
+            <max>3.5</max>
+            <resolution>0.015000</resolution>
+          </range>
+          <noise>
+            <type>gaussian</type>
+            <mean>0.0</mean>
+            <stddev>0.01</stddev>
+          </noise>
+        </ray>
+        <plugin name="scan" filename="libgazebo_ros_ray_sensor.so">
+          <ros>
+            <remapping>~/out:=scan</remapping>
+          </ros>
+          <output_type>sensor_msgs/LaserScan</output_type>
+          <frame_name>lidar_link</frame_name>
+        </plugin>
+      </sensor>
+    </link>
+    <!-- *********************** IMU SENSOR SETUP **************************  -->
+    <link name="imu_link">
+      <gravity>true</gravity>
+      <sensor name="bmb_imu" type="imu">
+        <always_on>true</always_on>
+        <update_rate>100</update_rate>
+        <visualize>true</visualize>
+        <imu>
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